File: battery-charging-experimentation.kicad_sch (KiCad schematic)
At the start: 23 parts, among them J1 USB_C_Receptacle_PowerOnly_6P, Q1 FS8205A, Q2 AO3415A, U2 DW01, U3 TP4056-42-ESOP8

Commit message: add switch to turn off pico
Parts:
- added SW1: MK-12C08-G1.5, easyeda2kicad:SW-SMD_DEALON_MK-12C08-G1.5, symbol easyeda2kicad:MK-12C08-G1.5
- Out1: footprint Connector_PinHeader_2.54mm:PinHeader_1x03_P2.54mm_Vertical -> Connector_PinHeader_2.54mm:PinHeader_1x04_P2.54mm_Vertical; symbol Connector:Conn_01x03_Pin -> Connector:Conn_01x04_Pin
- renumbered R_PR1 to RP1
Connections:
- net GND: now also Out1.2 (Pin_2), SW1.2; no longer Out1.1 (Pin_1)
- net VBUS: now also Out1.4 (Pin_4); no longer Out1.3 (Pin_3)
- net VBUS or BATT+: now also Out1.3 (Pin_3); no longer Out1.2 (Pin_2)
- new net: Out1.1 (Pin_1), SW1.1
- no-connect marks 34 -> 36
Changed lines of the file:
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@@
+	)
+	(no_connect
+		(at 200.66 144.78)
 	)
 	(no_connect
@@
 	)
 	(no_connect
+		(at 200.66 157.48)
+	)
+	(no_connect
 		(at 265.43 137.16)
 	)
@@
 	(wire
 		(pts
+			(xy 170.18 149.86) (xy 170.18 158.75)
+		)
+		(stroke
+			(width 0)
+			(type default)
+		)
+	)
+	(wire
+		(pts
 			(xy 87.63 170.18) (xy 91.44 170.18)
 		)
@@
 	(wire
 		(pts
+			(xy 173.99 154.94) (xy 171.45 154.94)
+		)
+		(stroke
+			(width 0)
+			(type default)
+		)
+	)
+	(wire
+		(pts
+			(xy 198.12 157.48) (xy 198.12 162.56)
+		)
+		(stroke
+			(width 0)
+			(type default)
+		)
+	)
+	(wire
+		(pts
 			(xy 142.24 106.68) (xy 123.19 106.68)
 		)
@@
 	(wire
 		(pts
+			(xy 170.18 149.86) (xy 173.99 149.86)
+		)
+		(stroke
+			(width 0)
+			(type default)
+		)
+	)
+	(wire
+		(pts
 			(xy 111.76 101.6) (xy 111.76 102.87)
 		)
@@
 	(wire
 		(pts
+			(xy 163.83 152.4) (xy 173.99 152.4)
+		)
+		(stroke
+			(width 0)
+			(type default)
+		)
+	)
+	(wire
+		(pts
 			(xy 58.42 146.05) (xy 130.81 146.05)
 		)
@@
 	(wire
 		(pts
-			(xy 170.18 153.67) (xy 170.18 158.75)
-		)
-		(stroke
-			(width 0)
-			(type default)
-		)
-	)
-	(wire
-		(pts
 			(xy 85.09 118.11) (xy 85.09 121.92)
 		)
@@
 	(wire
 		(pts
+			(xy 171.45 154.94) (xy 171.45 187.96)
+		)
+		(stroke
+			(width 0)
+			(type default)
+		)
+	)
+	(wire
+		(pts
 			(xy 93.98 124.46) (xy 93.98 121.92)
 		)
@@
 	(wire
 		(pts
+			(xy 195.58 161.29) (xy 195.58 157.48)
+		)
+		(stroke
+			(width 0)
+			(type default)
+		)
+	)
+	(wire
+		(pts
 			(xy 237.49 74.93) (xy 237.49 81.28)
 		)
@@
 	(wire
 		(pts
-			(xy 163.83 156.21) (xy 173.99 156.21)
+			(xy 173.99 157.48) (xy 173.99 161.29)
 		)
 		(stroke
@@
 	(wire
 		(pts
-			(xy 163.83 139.7) (xy 163.83 156.21)
+			(xy 173.99 161.29) (xy 195.58 161.29)
 		)
 		(stroke
@@
 	(wire
 		(pts
-			(xy 173.99 153.67) (xy 170.18 153.67)
-		)
-		(stroke
-			(width 0)
-			(type default)
-		)
-	)
-	(wire
-		(pts
 			(xy 160.02 158.75) (xy 160.02 170.18)
 		)
@@
 	(wire
 		(pts
-			(xy 173.99 187.96) (xy 171.45 187.96)
-		)
-		(stroke
-			(width 0)
-			(type default)
-		)
-	)
-	(wire
-		(pts
 			(xy 44.45 167.64) (xy 48.26 167.64)
 		)
@@
 	(wire
 		(pts
+			(xy 163.83 139.7) (xy 163.83 152.4)
+		)
+		(stroke
+			(width 0)
+			(type default)
+		)
+	)
+	(wire
+		(pts
 			(xy 109.22 102.87) (xy 111.76 102.87)
 		)
@@
 		(pts
 			(xy 143.51 151.13) (xy 140.97 151.13)
-		)
-		(stroke
-			(width 0)
-			(type default)
-		)
-	)
-	(wire
-		(pts
-			(xy 173.99 158.75) (xy 173.99 187.96)
 		)
 		(stroke
@@
 	)
 	(symbol
-		(lib_id "Connector:Conn_01x03_Pin")
-		(at 179.07 156.21 180)
+		(lib_id "Connector:Conn_01x04_Pin")
+		(at 179.07 154.94 180)
 		(unit 1)
 		(exclude_from_sim no)
@@
 		(dnp no)
 		(property "Reference" "Out1"
-			(at 179.07 147.32 0)
+			(at 179.07 146.05 0)
 			(effects
 				(font
@@
 		)
 		(property "Value" "Header"
-			(at 179.07 149.86 0)
-			(effects
-				(font
-					(size 1.27 1.27)
-				)
-			)
-		)
-		(property "Footprint" "Connector_PinHeader_2.54mm:PinHeader_1x03_P2.54mm_Vertical"
-			(at 179.07 156.21 0)
+			(at 179.07 148.59 0)
+			(effects
+				(font
+					(size 1.27 1.27)
+				)
+			)
+		)
+		(property "Footprint" "Connector_PinHeader_2.54mm:PinHeader_1x04_P2.54mm_Vertical"
+			(at 179.07 154.94 0)
 			(effects
 				(font
@@
 		)
 		(property "Datasheet" "~"
-			(at 179.07 156.21 0)
-			(effects
-				(font
-					(size 1.27 1.27)
-				)
-				(hide yes)
-			)
-		)
-		(property "Description" "Generic connector, single row, 01x03, script generated"
-			(at 179.07 156.21 0)
+			(at 179.07 154.94 0)
+			(effects
+				(font
+					(size 1.27 1.27)
+				)
+				(hide yes)
+			)
+		)
+		(property "Description" "Generic connector, single row, 01x04, script generated"
+			(at 179.07 154.94 0)
 			(effects
 				(font
@@
 		)
 		(property "LCSC Part" "C52016390"
-			(at 179.07 144.78 0)
+			(at 179.07 143.51 0)
 			(effects
 				(font
@@
 		)
 		(pin "3"
+		)
+		(pin "4"
 		)
 		(instances
@@
 		(on_board yes)
 		(dnp no)
-		(property "Reference" "R_PR1"
+		(property "Reference" "RP1"
 			(at 118.872 177.8 90)
 			(effects
@@
 			(project "battery-charging-experimentation"
 				(path "/b3c17f7d-b127-4261-827c-183ca4717040"
-					(reference "R_PR1")
+					(reference "RP1")
 					(unit 1)
 				)
@@
 	(symbol
 		(lib_id "power:GND")
+		(at 198.12 162.56 0)
+		(unit 1)
+		(exclude_from_sim no)
+		(in_bom yes)
+		(on_board yes)
+		(dnp no)
+		(fields_autoplaced yes)
+		(property "Reference" "#PWR08"
+			(at 198.12 168.91 0)
+			(effects
+				(font
+					(size 1.27 1.27)
+				)
+				(hide yes)
+			)
+		)
+		(property "Value" "GND"
+			(at 198.12 167.64 0)
+			(effects
+				(font
+					(size 1.27 1.27)
+				)
+			)
+		)
+		(property "Footprint" ""
+			(at 198.12 162.56 0)
+			(effects
+				(font
+					(size 1.27 1.27)
+				)
+				(hide yes)
+			)
+		)
+		(property "Datasheet" ""
+			(at 198.12 162.56 0)
+			(effects
+				(font
+					(size 1.27 1.27)
+				)
+				(hide yes)
+			)
+		)
+		(property "Description" "Power symbol creates a global label with name \"GND\" , ground"
+			(at 198.12 162.56 0)
+			(effects
+				(font
+					(size 1.27 1.27)
+				)
+				(hide yes)
+			)
+		)
+		(pin "1"
+		)
+		(instances
+			(project "battery-charging-experimentation"
+				(path "/b3c17f7d-b127-4261-827c-183ca4717040"
+					(reference "#PWR08")
+					(unit 1)
+				)
+			)
+		)
+	)
+	(symbol
+		(lib_id "power:GND")
 		(at 125.73 190.5 0)
 		(unit 1)
@@
 					(unit 1)
 				)
+			)
+		)
+	)
+	(symbol
+		(lib_id "easyeda2kicad:MK-12C08-G1.5")
+		(at 198.12 149.86 0)
+		(unit 1)
+		(exclude_from_sim no)
+		(in_bom yes)
+		(on_board yes)
+		(dnp no)
+		(fields_autoplaced yes)
+		(property "Reference" "SW1"
+			(at 204.47 147.3199 0)
+			(effects
+				(font
+					(size 1.27 1.27)
+				)
+				(justify left)
+			)
+		)
+		(property "Value" "MK-12C08-G1.5"
+			(at 204.47 149.8599 0)
+			(effects
+				(font
+					(size 1.27 1.27)
+				)
+				(justify left)
+			)
+		)
+		(property "Footprint" "easyeda2kicad:SW-SMD_DEALON_MK-12C08-G1.5"
+			(at 198.12 165.1 0)
+			(effects
+				(font
+					(size 1.27 1.27)
+				)
+				(hide yes)
+			)
+		)
+		(property "Datasheet" ""
+			(at 198.12 149.86 0)
+			(effects
+				(font
+					(size 1.27 1.27)
+				)
+				(hide yes)
+			)
+		)
+		(property "Description" ""
+			(at 198.12 149.86 0)
+			(effects
+				(font
+					(size 1.27 1.27)
+				)
+				(hide yes)
+			)
+		)
+		(property "LCSC Part" "C2904922"
+			(at 198.12 167.64 0)
+			(effects
+				(font
+					(size 1.27 1.27)
+				)
+				(hide yes)
+			)
+		)
+		(pin "4"
+		)
+		(pin "2"
+		)
+		(pin "1"
+		)
+		(pin "3"
+		)
+		(instances
+			(project ""
+				(path "/b3c17f7d-b127-4261-827c-183ca4717040"
+					(reference "SW1")
+					(unit 1)
+				)
